File: Hardware/Revision_B/geiger.kicad_pcb (KiCad board)
At the start: 2 copper layers, 123.1 x 31.9 mm, 26 parts, among them J1 I2C 5V, J2 I2C 3V3, J3 GND, U1 BSP125

Commit message: Hardware: add manufacturer part numbers to the BOMs and schematics
Rev A: update PARTS in gen_v110_bom_cpl.py and regenerate the BOM.
Rev B and Rev C: add a Part Number field to each schematic symbol and
push it to the PCB footprints.

Part number updates: C3 R75 -> R76, D3 BZX55 -> BZX79-B3V3,
R2-R5 MFR-25 -> RNV14, R6 RNV14FAL100K.

Also fixes the D3 part number CSV quoting, adds the missing tube-clip
and GND test-point rows, corrects the D3 and L1 values, and renames the
Rev C tube holder to SBM-19/20 to match the PCB.

Board geometry is unchanged.
Parts:
- D3: value BZX55 -> BZX79-B3V3
- L1: value L-11P -> 150mH
